File: HARDWARE/KICAD/ColorTemp.kicad_pcb (KiCad board)
At the start: 2 copper layers, 27.5 x 27.5 mm, 29 parts, among them J1 POWER, J2 EXPANSION, SW1 USER, SW2 ~{RESET}, U1 CH32V003F4U6, U2 MCP9700A

Commit message: Added QR code on PCB and links to sheets.
Parts:
- added G***: LOGO, LOGO, B.Cu at (150.0, 90.8)

Commit message: Had to replace de LED because it was not in Economic fabrication at JLC.
Parts:
- D1: value RGB -> WS2850B; footprint ColorTemp:LED_RGB_5050-6 -> ColorTemp:WS2850B
- turned D1 to 180 degrees
Connections:
- D1 pad 1: +5V -> LED BLUE
- D1 pad 2: +5V -> LED RED
- D1 pad 3: +5V -> LED GREEN
- D1 pad 4: LED BLUE -> +5V
- D1 pad 5: LED RED -> +5V
- D1 pad 6: LED GREEN -> +5V
